Commit message: URDF file - materials and Co

File: urdf/detectiBot.xacro (robot description, xacro)
@@ -1,6 +1,6 @@
 <?xml version="1.0" ?>
 <robot name="m2wr" xmlns:xacro="https://www.ros.org/wiki/xacro" >
- <xacro:include filename="$(find robot_urdf)/urdf/dbMaterials.xacro" />
- <xacro:include filename="$(find robot_urdf)/urdf/detectiBot.gazebo" />
+ <xacro:include filename="$(find explab_2nd)/urdf/materials.xacro" />
+ <xacro:include filename="$(find explab_2nd)/urdf/detectiBot.gazebo" />
  <xacro:macro name="cylinder_inertia" params="mass r l">
     <inertia ixx="${mass*(3*r*r+l*l)/12}" ixy = "0" ixz = "0"
@@ -42,5 +42,5 @@
     <pose>0 0 0.1 0 0 0</pose>
     <inertial>
-      <mass value="8"/>
+      <mass value="5"/>
       <origin rpy="0 0 0" xyz="0 0 0.1"/>
       <inertia ixx="0.0395416666667" ixy="0" ixz="0" iyy="0.106208333333" iyz="0" izz="0.106208333333"/>
@@ -115,5 +115,5 @@
   <link name="arm_base_link">
   	<inertial>
-  		<mass value="1.2"/>
+  		<mass value="0.1"/>
   		<origin xyz="0 0 0" rpy="0 0 0" />
   		<inertia ixx="0.0000416666667" ixy="0" ixz="0" iyy="0.0000416666667" iyz="0" izz="0.0000416666667"/>
@@ -140,18 +140,18 @@
   <link name="arm_link_01">
   	<inertial>
-  		<mass value="0.03"/>
-  		<origin xyz="0 0 0" rpy="0 0 0" />
-  		<inertia ixx="0.000010279" ixy="0" ixz="0" iyy="0.000010279" iyz="0" izz="0.000007225"/>
-  	</inertial>
-  	<collision>
-  	  <origin xyz="0 0 0.3" rpy="0 0 0"/>
-      <geometry>
-        <cylinder radius="0.04" length="0.3"/>
-      </geometry>
-  	</collision>
-  	<visual>
-  	  <origin xyz="0 0 3" rpy="0 0 0"/>
-      <geometry>
-        <cylinder radius="0.04" length="0.3"/>
+  		<mass value="0.025"/>
+  		<origin xyz="0 0 0" rpy="0 0 0" />
+  		<inertia ixx="0.000010279" ixy="0" ixz="0" iyy="0.000010279" iyz="0" izz="0.000007225"/>
+  	</inertial>
+  	<collision>
+  	  <origin xyz="0 0 0" rpy="0 0 0"/>
+      <geometry>
+        <cylinder radius="0.04" length="0.08"/>
+      </geometry>
+  	</collision>
+  	<visual>
+  	  <origin xyz="0 0 0" rpy="0 0 0"/>
+      <geometry>
+        <cylinder radius="0.04" length="0.08"/>
       </geometry>
       <material name="red" />
@@ -167,18 +167,18 @@
     <link name="arm_link_02">
   	<inertial>
-  		<mass value="0.02"/>
-  		<origin xyz="0 0 0" rpy="0 0 0" />
-  		<inertia ixx="0.000010279" ixy="0" ixz="0" iyy="0.000010279" iyz="0" izz="0.000007225"/>
-  	</inertial>
-  	<collision>
-  	  <origin xyz="0 0 0.20" rpy="0 0 0"/>
-      <geometry>
-        <cylinder radius="0.04" length="0.08"/>
-      </geometry>
-  	</collision>
-  	<visual>
-  	  <origin xyz="0 0 0.20" rpy="0 0 0"/>
-      <geometry>
-        <cylinder radius="0.04" length="0.3"/>
+  		<mass value="0.025"/>
+  		<origin xyz="0 0 0" rpy="0 0 0" />
+  		<inertia ixx="0.000010279" ixy="0" ixz="0" iyy="0.000010279" iyz="0" izz="0.000007225"/>
+  	</inertial>
+  	<collision>
+  	  <origin xyz="0 0 0.04" rpy="0 0 0"/>
+      <geometry>
+        <cylinder radius="0.04" length="0.08"/>
+      </geometry>
+  	</collision>
+  	<visual>
+  	  <origin xyz="0 0 0.04" rpy="0 0 0"/>
+      <geometry>
+        <cylinder radius="0.04" length="0.08"/>
       </geometry>
       <material name="red" />
@@ -194,5 +194,5 @@
       <link name="arm_link_03">
   	<inertial>
-  		<mass value="0.02"/>
+  		<mass value="0.025"/>
   		<origin xyz="0 0 0" rpy="0 0 0" />
   		<inertia ixx="0.000010279" ixy="0" ixz="0" iyy="0.000010279" iyz="0" izz="0.000007225"/>
@@ -246,24 +246,4 @@
   	<child link="arm_link_04"/>
   </joint>
-  <link name="cluedo_link">
-  	<inertial>
-  		<mass value="0.004"/>
-  		<origin xyz="0 0 0" rpy="0 0 0" />
-  		<inertia ixx="0.000010279" ixy="0" ixz="0" iyy="0.000010279" iyz="0" izz="0.000007225"/>
-  	</inertial>
-  	<collision>
-  	  <origin xyz="0 0 0.04" rpy="0 0 1.57"/>
-      <geometry>
-        <box size="0.04 0.3 0.1"/>
-      </geometry>
-  	</collision>
-  	<visual>
-  	  <origin xyz="0 0 0.04" rpy="0 0 1.57"/>
-      <geometry>
-        <box size="0.034 0.2 0.08"/>
-      </geometry>
-      <material name="red" />
-  	</visual>
-  </link>
 <link name="right_grip_link">
   	<inertial>

Commit message: detectiBot model added

File: urdf/detectiBot.xacro (robot description, xacro)
@@ -1,6 +1,19 @@
 <?xml version="1.0" ?>
-<robot name="m2wr" xmlns:xacro="https://www.ros.org/wiki/xacro" >
+<robot name="detectiBot" xmlns:xacro="https://www.ros.org/wiki/xacro" >
+<!-- =================================================================================== -->
+<!-- |                                 detectiBot model                                | -->
+<!-- |                             Experimental robotics lab                           | -->
+<!-- =================================================================================== -->
+<!-- ==================================== Xacro include ============================================ -->
  <xacro:include filename="$(find explab_2nd)/urdf/materials.xacro" />
  <xacro:include filename="$(find explab_2nd)/urdf/detectiBot.gazebo" />
+<!-- ================================== Properties' list ============================================ -->
+<!-- ======================== All units in m-kg-s-radians unit system =============================== -->
+  <xacro:property name="M_PI" value="3.1415926535897931" />
+  <xacro:property name="M_PI_2" value="1.570796327" />
+  <xacro:property name="DEG_TO_RAD" value="0.017453293" />
+  <xacro:property name="arm_link_mass" value="0.025"/>
+  <xacro:property name="base_link_mass" value="5"/>
+<!-- ================================== Xacro definitions ========================================== -->
  <xacro:macro name="cylinder_inertia" params="mass r l">
     <inertia ixx="${mass*(3*r*r+l*l)/12}" ixy = "0" ixz = "0"
@@ -38,4 +51,5 @@
       </joint>
     </xacro:macro>
+<!-- ======================================== Link  ================================================ -->
   <link name="base_link">
     <!-- pose and inertial -->
@@ -46,4 +60,5 @@
       <inertia ixx="0.0395416666667" ixy="0" ixz="0" iyy="0.106208333333" iyz="0" izz="0.106208333333"/>
     </inertial>
+    <!-- chassis collision -->
     <collision name="collision_chassis">
       <geometry>
@@ -58,5 +73,5 @@
       <material name="blue"/>
     </visual>
-    <!-- caster front -->
+    <!-- caster front collision -->
     <collision name="caster_front_collision">
       <origin rpy=" 0 0 0" xyz="0.35 0 -0.05"/>
@@ -81,10 +96,11 @@
       </geometry>
     </visual>
-    </link>
-  <!-- Create wheels -->
+  </link>
+<!-- ==================================== Create wheels ============================================ -->
   <xacro:link_wheel name="link_right_wheel" />
   <xacro:link_wheel name="link_left_wheel" />
   <xacro:joint_wheel name="joint_right_wheel"  child="link_right_wheel"  origin_xyz="-0.05 0.15 0"  />
   <xacro:joint_wheel name="joint_left_wheel"   child="link_left_wheel"   origin_xyz="-0.05 -0.15 0"  />
+<!-- ======================================== Link  ================================================ -->
    <link name="laser">
     <inertial>
@@ -107,4 +123,5 @@
     </collision>
   </link>
+<!-- ======================================== Joint  =============================================== -->
   <joint name="joint_laser" type="fixed">
     <origin xyz="0.15 0 0.05" rpy="0 0 0"/>
@@ -112,5 +129,6 @@
     <child link="laser"/>
   </joint>
-<!--arm definition -->
+<!-- ======================================== Link  ================================================ -->
+<!-- ==================================== arm definition =========================================== -->
   <link name="arm_base_link">
   	<inertial>
@@ -138,4 +156,5 @@
   	<child link="arm_base_link"/>
   </joint>
+<!-- ======================================== Link  ================================================ -->
   <link name="arm_link_01">
   	<inertial>
@@ -158,4 +177,5 @@
   	</visual>
   </link>
+<!-- ======================================== Joint  =============================================== -->
   <joint name="arm_joint_01" type="revolute">
   	<axis xyz="0 0 1"/>
@@ -165,4 +185,5 @@
   	<child link="arm_link_01"/>
   </joint>
+<!-- ======================================== Link  ================================================ -->
     <link name="arm_link_02">
   	<inertial>
@@ -185,4 +206,5 @@
   	</visual>
   </link>
+<!-- ======================================== Joint  =============================================== -->
   <joint name="arm_joint_02" type="revolute">
   	<axis xyz="1 0 0"/>
@@ -192,4 +214,5 @@
   	<child link="arm_link_02"/>
   </joint>
+<!-- ======================================== Link  ================================================ -->
       <link name="arm_link_03">
   	<inertial>
@@ -212,4 +235,5 @@
   	</visual>
   </link>
+<!-- ======================================== Joint  =============================================== -->
   <joint name="arm_joint_03" type="revolute">
   	<axis xyz="1 0 0"/>
@@ -219,5 +243,6 @@
   	<child link="arm_link_03"/>
   </joint>
-    <link name="arm_link_04">
+<!-- ======================================== Link  ================================================ -->
+    <link name="cluedo_link">
   	<inertial>
   		<mass value="0.025"/>
@@ -239,4 +264,5 @@
   	</visual>
   </link>
+<!-- ======================================== Joint  =============================================== -->
   <joint name="arm_joint_04" type="revolute">
   	<axis xyz="1 0 0"/>
@@ -244,6 +270,7 @@
   	<origin rpy="0 0 0" xyz="0 0 0.08"/>
   	<parent link="arm_link_03"/>
-  	<child link="arm_link_04"/>
-  </joint>
+  	<child link="cluedo_link"/>
+  </joint>
+<!-- ======================================== Link  ================================================ -->
 <link name="right_grip_link">
   	<inertial>
@@ -266,11 +293,13 @@
   	</visual>
   </link>
+<!-- ======================================== Joint  =============================================== -->
   <joint name="right_grip_joint" type="prismatic">
   	<axis xyz="1 0 0"/>
   	<limit effort="1000.0" lower="-0.04" upper="0.035" velocity="6.5"/>
   	<origin rpy="0 0 0" xyz="-0.015 0 0.0"/>
-  	<parent link="arm_link_04"/>
+  	<parent link="cluedo_link"/>
   	<child link="right_grip_link"/>
   </joint>
+<!-- ======================================== Link  ================================================ -->
   <link name="left_grip_link">
   	<inertial>
@@ -293,9 +322,10 @@
   	</visual>
   </link>
+<!-- ======================================== Joint  =============================================== -->
   <joint name="left_grip_joint" type="prismatic">
   	<axis xyz="1 0 0"/>
   	<limit effort="1000.0" upper="0.04" lower="-0.035" velocity="6.5"/>
   	<origin rpy="0 0 0" xyz="-0.015 0 0.0"/>
-  	<parent link="arm_link_04"/>
+  	<parent link="cluedo_link"/>
   	<child link="left_grip_link"/>
   </joint>

File: urdf/materials.xacro (robot description, xacro)
@@ -1,6 +1,12 @@
 <?xml version="1.0" ?>
 <robot name="detectibot" xmlns:xacro="https://www.ros.org/wiki/xacro" >
+  <material name="neongreen" >
+    <color rgba="0.047058823529411764 1.0 0.047058823529411764 1.0" />
+  </material>
   <material name="black">
     <color rgba="0.0 0.0 0.0 1.0"/>
+  </material>
+  <material name="acidgreen" >
+    <color rgba="0.5607843137254902 0.996078431372549 0.03529411764705882 1.0" />
   </material>
   <material name="blue">
@@ -10,6 +16,12 @@
     <color rgba="0.0 0.8 0.0 1.0"/>
   </material>
+  <material name="ocre" >
+    <color rgba="0.7764705882352941 0.611764705882353 0.01568627450980392 1.0" />
+  </material>
   <material name="grey">
     <color rgba="0.2 0.2 0.2 1.0"/>
+  </material>
+  <material name="bruise" >
+    <color rgba="0.49411764705882355 0.25098039215686274 0.44313725490196076 1.0" />
   </material>
   <material name="orange">
@@ -18,4 +30,10 @@
   <material name="brown">
     <color rgba="0.870588235294 0.811764705882 0.764705882353 1.0"/>
+  </material>
+  <material name="burgundy" >
+    <color rgba="0.3803921568627451 0.0 0.13725490196078433 1.0" />
+  </material>
+  <material name="dusk" >
+    <color rgba="0.3058823529411765 0.32941176470588235 0.5058823529411764 1.0" />
   </material>
   <material name="red">

Commit message: robot description

File: urdf/detectiBot.xacro (robot description, xacro)
@@ -10,9 +10,16 @@
 <!-- ================================== Properties' list ============================================ -->
 <!-- ======================== All units in m-kg-s-radians unit system =============================== -->
+<!-- math and conversion  -->
   <xacro:property name="M_PI" value="3.1415926535897931" />
   <xacro:property name="M_PI_2" value="1.570796327" />
   <xacro:property name="DEG_TO_RAD" value="0.017453293" />
+<!-- mass  -->
   <xacro:property name="arm_link_mass" value="0.025"/>
-  <xacro:property name="base_link_mass" value="5"/>
+  <xacro:property name="base_link_mass" value="1"/>
+  <xacro:property name="gripper_link_mass" value="0.2"/>
+<!-- lenght -->
+  <xacro:property name="arm_link_01_lenght" value="0.3"/>
+  <xacro:property name="arm_link_02_lenght" value="0.3"/>
+  <xacro:property name="arm_link_03_lenght" value="0.3"/>
 <!-- ================================== Xacro definitions ========================================== -->
  <xacro:macro name="cylinder_inertia" params="mass r l">
@@ -56,5 +63,5 @@
     <pose>0 0 0.1 0 0 0</pose>
     <inertial>
-      <mass value="5"/>
+      <mass value="base_link_mass"/>
       <origin rpy="0 0 0" xyz="0 0 0.1"/>
       <inertia ixx="0.0395416666667" ixy="0" ixz="0" iyy="0.106208333333" iyz="0" izz="0.106208333333"/>
@@ -151,4 +158,5 @@
   	</visual>
   </link>
+<!-- ======================================== Joint  =============================================== -->
   <joint name="arm_base_to_base" type="fixed">
   	<origin rpy="0 0 0" xyz="0 0 0.085"/>
@@ -159,18 +167,18 @@
   <link name="arm_link_01">
   	<inertial>
-  		<mass value="0.025"/>
-  		<origin xyz="0 0 0" rpy="0 0 0" />
-  		<inertia ixx="0.000010279" ixy="0" ixz="0" iyy="0.000010279" iyz="0" izz="0.000007225"/>
-  	</inertial>
-  	<collision>
-  	  <origin xyz="0 0 0" rpy="0 0 0"/>
-      <geometry>
-        <cylinder radius="0.04" length="0.08"/>
-      </geometry>
-  	</collision>
-  	<visual>
-  	  <origin xyz="0 0 0" rpy="0 0 0"/>
-      <geometry>
-        <cylinder radius="0.04" length="0.08"/>
+  		<mass value="${arm_link_mass}"/>
+  		<origin xyz="0 0 ${arm_link_01_lenght/2}" rpy="0 0 0" />
+  		<inertia ixx="0.000010279" ixy="0" ixz="0" iyy="0.000010279" iyz="0" izz="0.000007225"/>
+  	</inertial>
+  	<collision>
+  	  <origin xyz="0 0 ${arm_link_01_lenght/2}" rpy="0 0 0"/>
+      <geometry>
+        <cylinder radius="0.04" length="${arm_link_01_lenght}"/>
+      </geometry>
+  	</collision>
+  	<visual>
+  	  <origin xyz="0 0 ${arm_link_01_lenght/2}" rpy="0 0 0"/>
+      <geometry>
+        <cylinder radius="0.04" length="${arm_link_01_lenght}"/>
       </geometry>
       <material name="red" />
@@ -181,5 +189,5 @@
   	<axis xyz="0 0 1"/>
   	<limit effort="1000.0" lower="-3.14" upper="3.14" velocity="0.2"/>
-  	<origin rpy="0 0 0" xyz="0 0 0.09"/>
+  	<origin rpy="0 0 0" xyz="0 0 ${arm_link_01_lenght}"/>
   	<parent link="arm_base_link"/>
   	<child link="arm_link_01"/>
@@ -188,18 +196,18 @@
     <link name="arm_link_02">
   	<inertial>
-  		<mass value="0.025"/>
-  		<origin xyz="0 0 0" rpy="0 0 0" />
-  		<inertia ixx="0.000010279" ixy="0" ixz="0" iyy="0.000010279" iyz="0" izz="0.000007225"/>
-  	</inertial>
-  	<collision>
-  	  <origin xyz="0 0 0.04" rpy="0 0 0"/>
-      <geometry>
-        <cylinder radius="0.04" length="0.08"/>
-      </geometry>
-  	</collision>
-  	<visual>
-  	  <origin xyz="0 0 0.04" rpy="0 0 0"/>
-      <geometry>
-        <cylinder radius="0.04" length="0.08"/>
+  		<mass value="${arm_link_mass}"/>
+  		<origin xyz="0 0 ${arm_link_02_lenght/2}" rpy="0 0 0" />
+  		<inertia ixx="0.000010279" ixy="0" ixz="0" iyy="0.000010279" iyz="0" izz="0.000007225"/>
+  	</inertial>
+  	<collision>
+  	  <origin xyz="0 0 ${arm_link_02_lenght/2}" rpy="0 0 0"/>
+      <geometry>
+        <cylinder radius="0.04" length="${arm_link_02_lenght}"/>
+      </geometry>
+  	</collision>
+  	<visual>
+  	  <origin xyz="0 0 ${arm_link_02_lenght/2}" rpy="0 0 0"/>
+      <geometry>
+        <cylinder radius="0.04" length="${arm_link_02_lenght}"/>
       </geometry>
       <material name="red" />
@@ -210,5 +218,5 @@
   	<axis xyz="1 0 0"/>
   	<limit effort="1000.0" lower="-1.8" upper="1.8" velocity="0.2"/>
-  	<origin rpy="0 0 0" xyz="0 0 0.04"/>
+  	<origin rpy="0 0 0" xyz="0 0 ${arm_link_02_lenght/2}"/>
   	<parent link="arm_link_01"/>
   	<child link="arm_link_02"/>
@@ -217,18 +225,18 @@
       <link name="arm_link_03">
   	<inertial>
-  		<mass value="0.025"/>
-  		<origin xyz="0 0 0" rpy="0 0 0" />
-  		<inertia ixx="0.000010279" ixy="0" ixz="0" iyy="0.000010279" iyz="0" izz="0.000007225"/>
-  	</inertial>
-  	<collision>
-  	  <origin xyz="0 0 0.04" rpy="0 0 0"/>
-      <geometry>
-        <cylinder radius="0.04" length="0.08"/>
-      </geometry>
-  	</collision>
-  	<visual>
-  	  <origin xyz="0 0 0.04" rpy="0 0 0"/>
-      <geometry>
-        <cylinder radius="0.04" length="0.08"/>
+  		<mass value="${arm_link_mass}"/>
+  		<origin xyz="0 0 ${arm_link_03_lenght/2}" rpy="0 0 0" />
+  		<inertia ixx="0.000010279" ixy="0" ixz="0" iyy="0.000010279" iyz="0" izz="0.000007225"/>
+  	</inertial>
+  	<collision>
+  	  <origin xyz="0 0 ${arm_link_03_lenght/2}" rpy="0 0 0"/>
+      <geometry>
+        <cylinder radius="0.04" length="${arm_link_03_lenght}"/>
+      </geometry>
+  	</collision>
+  	<visual>
+  	  <origin xyz="0 0 ${arm_link_03_lenght/2}" rpy="0 0 0"/>
+      <geometry>
+        <cylinder radius="0.04" length="${arm_link_03_lenght}"/>
       </geometry>
       <material name="red" />
@@ -239,5 +247,5 @@
   	<axis xyz="1 0 0"/>
   	<limit effort="1000.0" lower="-1.8" upper="1.8" velocity="0.2"/>
-  	<origin rpy="0 0 0" xyz="0 0 0.08"/>
+  	<origin rpy="0 0 0" xyz="0 0 ${arm_link_03_lenght/2}"/>
   	<parent link="arm_link_02"/>
   	<child link="arm_link_03"/>
@@ -247,9 +255,9 @@
   	<inertial>
   		<mass value="0.025"/>
-  		<origin xyz="0 0 0" rpy="0 0 0" />
-  		<inertia ixx="0.000010279" ixy="0" ixz="0" iyy="0.000010279" iyz="0" izz="0.000007225"/>
-  	</inertial>
-  	<collision>
-  	  <origin xyz="0 0 0.04" rpy="0 0 1.57"/>
+  		<origin xyz="0 0 ${cluedo_link_lenght/2}" rpy="0 0 0" />
+  		<inertia ixx="0.000010279" ixy="0" ixz="0" iyy="0.000010279" iyz="0" izz="0.000007225"/>
+  	</inertial>
+  	<collision>
+  	  <origin xyz="0 0 ${cluedo_link_lenght/2}" rpy="0 0 1.57"/>
       <geometry>
         <box size="0.034 0.2 0.08"/>
@@ -257,5 +265,5 @@
   	</collision>
   	<visual>
-  	  <origin xyz="0 0 0.04" rpy="0 0 1.57"/>
+  	  <origin xyz="0 0 ${cluedo_link_lenght/2}" rpy="0 0 1.57"/>
       <geometry>
         <box size="0.034 0.2 0.08"/>
@@ -268,5 +276,5 @@
   	<axis xyz="1 0 0"/>
   	<limit effort="1000.0" lower="-1.8" upper="1.8" velocity="0.5"/>
-  	<origin rpy="0 0 0" xyz="0 0 0.08"/>
+  	<origin rpy="0 0 0" xyz="0 0 ${cluedo_link_lenght/2}"/>
   	<parent link="arm_link_03"/>
   	<child link="cluedo_link"/>
@@ -330,3 +338,64 @@
   	<child link="left_grip_link"/>
   </joint>
+<!-- ===================================== Transmission  ============================================ -->
+<transmission name="arm_joint_01_trans">
+	<type>transmission_interface/SimpleTransmission</type>
+	<joint name="arm_joint_01">
+		<hardwareInterface>hardware_interface/EffortJointInterface</hardwareInterface>
+	</joint>
+	<actuator name="motor1">
+		<hardwareInterface>hardware_interface/EffortJointInterface</hardwareInterface>
+		<mechanicalInterface>1</mechanicalInterface>
+	</actuator>
+</transmission>
+<transmission name="arm_joint_02_trans">
+	<type>transmission_interface/SimpleTransmission</type>
+	<joint name="arm_joint_02">
+		<hardwareInterface>hardware_interface/EffortJointInterface</hardwareInterface>
+	</joint>
+	<actuator name="motor2">
+		<hardwareInterface>hardware_interface/EffortJointInterface</hardwareInterface>
+		<mechanicalInterface>1</mechanicalInterface>
+	</actuator>
+</transmission>
+<transmission name="arm_joint_03_trans">
+	<type>transmission_interface/SimpleTransmission</type>
+	<joint name="arm_joint_03">
+		<hardwareInterface>hardware_interface/EffortJointInterface</hardwareInterface>
+	</joint>
+	<actuator name="motor3">
+		<hardwareInterface>hardware_interface/EffortJointInterface</hardwareInterface>
+		<mechanicalInterface>1</mechanicalInterface>
+	</actuator>
+</transmission>
+<transmission name="arm_joint_04_trans">
+	<type>transmission_interface/SimpleTransmission</type>
+	<joint name="arm_joint_04">
+		<hardwareInterface>hardware_interface/EffortJointInterface</hardwareInterface>
+	</joint>
+	<actuator name="motor4">
+		<hardwareInterface>hardware_interface/EffortJointInterface</hardwareInterface>
+		<mechanicalInterface>1</mechanicalInterface>
+	</actuator>
+</transmission>
+<transmission name="left_grip_trans">
+	<type>transmission_interface/SimpleTransmission</type>
+	<joint name="left_grip_joint">
+		<hardwareInterface>hardware_interface/EffortJointInterface</hardwareInterface>
+	</joint>
+	<actuator name="motor5">
+		<hardwareInterface>hardware_interface/EffortJointInterface</hardwareInterface>
+		<mechanicalInterface>1</mechanicalInterface>
+	</actuator>
+</transmission>
+<transmission name="right_grip_trans">
+	<type>transmission_interface/SimpleTransmission</type>
+	<joint name="right_grip_joint">
+		<hardwareInterface>hardware_interface/EffortJointInterface</hardwareInterface>
+	</joint>
+	<actuator name="motor6">
+		<hardwareInterface>hardware_interface/EffortJointInterface</hardwareInterface>
+		<mechanicalInterface>1</mechanicalInterface>
+	</actuator>
+</transmission>
 </robot>
