Commit message: some adjustments to the robot model

File: urdf/detectiBot.xacro (robot description, xacro)
@@ -16,5 +16,5 @@
 <!-- mass  -->
   <xacro:property name="arm_link_mass" value="0.025"/>
-  <xacro:property name="base_link_mass" value="1"/>
+  <xacro:property name="base_link_mass" value="0.5"/>
   <xacro:property name="gripper_link_mass" value="0.2"/>
 <!-- lenght -->
@@ -22,4 +22,6 @@
   <xacro:property name="arm_link_02_lenght" value="0.3"/>
   <xacro:property name="arm_link_03_lenght" value="0.3"/>
+  <xacro:property name="cluedo_link_lenght" value="0.3"/>
+  <xacro:property name="err" value="-0.2"/>
 <!-- ================================== Xacro definitions ========================================== -->
  <xacro:macro name="cylinder_inertia" params="mass r l">
@@ -63,5 +65,5 @@
     <pose>0 0 0.1 0 0 0</pose>
     <inertial>
-      <mass value="base_link_mass"/>
+      <mass value="${base_link_mass}"/>
       <origin rpy="0 0 0" xyz="0 0 0.1"/>
       <inertia ixx="0.0395416666667" ixy="0" ixz="0" iyy="0.106208333333" iyz="0" izz="0.106208333333"/>
@@ -147,5 +149,5 @@
   	  <origin xyz="0 0 0" rpy="0 0 0"/>
       <geometry>
-        <box size="0.1 0.1 0.1"/>
+        <box size="0.1 0.1 0.15"/>
       </geometry>
   	</collision>
@@ -153,7 +155,7 @@
   	  <origin xyz="0 0 0" rpy="0 0 0"/>
       <geometry>
-        <box size="0.1 0.1 0.1"/>
-      </geometry>
-      <material name="red" />
+        <box size="0.1 0.1 0.2"/>
+      </geometry>
+      <material name="white" />
   	</visual>
   </link>
@@ -189,5 +191,5 @@
   	<axis xyz="0 0 1"/>
   	<limit effort="1000.0" lower="-3.14" upper="3.14" velocity="0.2"/>
-  	<origin rpy="0 0 0" xyz="0 0 ${arm_link_01_lenght}"/>
+  	<origin rpy="0 0 0" xyz="0 0 ${arm_link_01_lenght/2 -0.1}"/>
   	<parent link="arm_base_link"/>
   	<child link="arm_link_01"/>
@@ -288,5 +290,5 @@
   	</inertial>
   	<collision>
-  	  <origin xyz="-0.032 0.048 0.04" rpy="0 3.1415 -1.57"/>
+  	  <origin xyz="-0.032 0.048 0.15" rpy="0 3.1415 -1.57"/>
       <geometry>
         <box size="0.06 0.02 0.08"/>
@@ -294,5 +296,5 @@
   	</collision>
   	<visual>
-  	  <origin xyz="-0.032 0.048 0.04" rpy="0 3.1415 -1.57"/>
+  	  <origin xyz="-0.032 0.048 0.15" rpy="0 3.1415 -1.57"/>
       <geometry>
         <box size="0.06 0.02 0.08"/>
@@ -317,5 +319,5 @@
   	</inertial>
   	<collision>
-  	  <origin xyz="0.06 0.048 0.04" rpy="0 3.1415 -1.57"/>
+  	  <origin xyz="0.06 0.048 0.15" rpy="0 3.1415 -1.57"/>
       <geometry>
         <box size="0.06 0.02 0.08"/>
@@ -323,5 +325,5 @@
   	</collision>
   	<visual>
-  	  <origin xyz="0.06 0.048 0.04" rpy="0 3.1415 -1.57"/>
+  	  <origin xyz="0.06 0.048 0.15" rpy="0 3.1415 -1.57"/>
       <geometry>
         <box size="0.06 0.02 0.08"/>
