Commit message: model updated

File: urdf/detectiBot.urdf (robot description, URDF)
Before this commit: robot detectiBot, 11 links, 10 joints
Joints:
- joint arm_joint_02: origin xyz=0 0 0.15 rpy=0 0 0 -> xyz=0 0 0.3 rpy=0 0 0
- joint arm_joint_03: origin xyz=0 0 0.15 rpy=0 0 0 -> xyz=0 0 0.3 rpy=0 0 0
- joint arm_joint_04: type revolute -> fixed
- joint left_grip_joint: origin xyz=-0.015 0 0.0 rpy=0 0 0 -> xyz=-0.015 0 0.15 rpy=0 0 0
- joint right_grip_joint: origin xyz=-0.015 0 0.0 rpy=0 0 0 -> xyz=-0.015 0 0.15 rpy=0 0 0

File: urdf/detectiBot.xacro (robot description, xacro)
@@ -220,5 +220,5 @@
   	<axis xyz="1 0 0"/>
   	<limit effort="1000.0" lower="-1.8" upper="1.8" velocity="0.2"/>
-  	<origin rpy="0 0 0" xyz="0 0 ${arm_link_02_lenght/2}"/>
+  	<origin rpy="0 0 0" xyz="0 0 ${arm_link_02_lenght/2 + 0.15}"/>
   	<parent link="arm_link_01"/>
   	<child link="arm_link_02"/>
@@ -249,5 +249,5 @@
   	<axis xyz="1 0 0"/>
   	<limit effort="1000.0" lower="-1.8" upper="1.8" velocity="0.2"/>
-  	<origin rpy="0 0 0" xyz="0 0 ${arm_link_03_lenght/2}"/>
+  	<origin rpy="0 0 0" xyz="0 0 ${arm_link_03_lenght/2 + 0.15}"/>
   	<parent link="arm_link_02"/>
   	<child link="arm_link_03"/>
@@ -275,5 +275,5 @@
   </link>
 <!-- ======================================== Joint  =============================================== -->
-  <joint name="arm_joint_04" type="revolute">
+  <joint name="arm_joint_04" type="fixed">
   	<axis xyz="1 0 0"/>
   	<limit effort="1000.0" lower="-1.8" upper="1.8" velocity="0.5"/>
@@ -290,5 +290,5 @@
   	</inertial>
   	<collision>
-  	  <origin xyz="-0.032 0.048 0.15" rpy="0 3.1415 -1.57"/>
+  	  <origin xyz="-0.032 0.048 0.0" rpy="0 3.1415 -1.57"/>
       <geometry>
         <box size="0.06 0.02 0.08"/>
@@ -296,5 +296,5 @@
   	</collision>
   	<visual>
-  	  <origin xyz="-0.032 0.048 0.15" rpy="0 3.1415 -1.57"/>
+  	  <origin xyz="-0.032 0.048 0.0" rpy="0 3.1415 -1.57"/>
       <geometry>
         <box size="0.06 0.02 0.08"/>
@@ -307,5 +307,5 @@
   	<axis xyz="1 0 0"/>
   	<limit effort="1000.0" lower="-0.04" upper="0.035" velocity="6.5"/>
-  	<origin rpy="0 0 0" xyz="-0.015 0 0.0"/>
+  	<origin rpy="0 0 0" xyz="-0.015 0 0.15"/>
   	<parent link="cluedo_link"/>
   	<child link="right_grip_link"/>
@@ -319,5 +319,5 @@
   	</inertial>
   	<collision>
-  	  <origin xyz="0.06 0.048 0.15" rpy="0 3.1415 -1.57"/>
+  	  <origin xyz="0.06 0.048 0.0" rpy="0 3.1415 -1.57"/>
       <geometry>
         <box size="0.06 0.02 0.08"/>
@@ -325,5 +325,5 @@
   	</collision>
   	<visual>
-  	  <origin xyz="0.06 0.048 0.15" rpy="0 3.1415 -1.57"/>
+  	  <origin xyz="0.06 0.048 0.0" rpy="0 3.1415 -1.57"/>
       <geometry>
         <box size="0.06 0.02 0.08"/>
@@ -336,5 +336,5 @@
   	<axis xyz="1 0 0"/>
   	<limit effort="1000.0" upper="0.04" lower="-0.035" velocity="6.5"/>
-  	<origin rpy="0 0 0" xyz="-0.015 0 0.0"/>
+  	<origin rpy="0 0 0" xyz="-0.015 0 0.15"/>
   	<parent link="cluedo_link"/>
   	<child link="left_grip_link"/>

Commit message: last verison of robot model + motors_configuration file

File: urdf/detectiBot.urdf (robot description, URDF)
Before this commit: robot detectiBot, 11 links, 10 joints
Joints:
- joint arm_joint_04: type fixed -> revolute

File: urdf/detectiBot.xacro (robot description, xacro)
@@ -275,5 +275,5 @@
   </link>
 <!-- ======================================== Joint  =============================================== -->
-  <joint name="arm_joint_04" type="fixed">
+  <joint name="arm_joint_04" type="revolute">
   	<axis xyz="1 0 0"/>
   	<limit effort="1000.0" lower="-1.8" upper="1.8" velocity="0.5"/>
